Commit message: regenerate urdf file from xacro file

File: urdf/mini_pupper_description.urdf (robot description, URDF)
Before this commit: robot mini_pupper_description, 38 links, 37 joints
Links:
- added link base_inertia, mass 0.7
- link base_link: mass 0.7 -> None; geometry collision mesh filename=file:///home/cullen/ros2_ws/install/mini_pupper_description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; visual mesh filename=file:///home/cullen/ros2_ws/install/mini_pupper_description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
- link camera_link: geometry collision box size=0.02505 0.09 0.025; visual mesh filename=file:///home/cullen/ros2_ws/install/mini_pupper_description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
- link lb1: geometry collision mesh filename=file:///home/cullen/ros2_ws/install/mini_pupper_description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; visual mesh filename=file:///home/cullen/ros2_ws/install/mini_pupper_description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
- link lb2: geometry collision mesh filename=file:///home/cullen/ros2_ws/install/mini_pupper_description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; visual mesh filename=file:///home/cullen/ros2_ws/install/mini_pupper_description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
- link lb3: geometry collision mesh filename=file:///home/cullen/ros2_ws/install/mini_pupper_description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; visual mesh filename=file:///home/cullen/ros2_ws/install/mini_pupper_description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
- link lbfoot: geometry collision mesh filename=file:///home/cullen/ros2_ws/install/mini_pupper_description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; visual mesh filename=file:///home/cullen/ros2_ws/install/mini_pupper_description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
- link lf1: geometry collision mesh filename=file:///home/cullen/ros2_ws/install/mini_pupper_description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; visual mesh filename=file:///home/cullen/ros2_ws/install/mini_pupper_description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
- link lf2: geometry collision mesh filename=file:///home/cullen/ros2_ws/install/mini_pupper_description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; visual mesh filename=file:///home/cullen/ros2_ws/install/mini_pupper_description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
- link lf3: geometry collision mesh filename=file:///home/cullen/ros2_ws/install/mini_pupper_description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; visual mesh filename=file:///home/cullen/ros2_ws/install/mini_pupper_description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
- link lffoot: geometry collision mesh filename=file:///home/cullen/ros2_ws/install/mini_pupper_description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; visual mesh filename=file:///home/cullen/ros2_ws/install/mini_pupper_description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
- link lidar: geometry collision mesh filename=file:///home/cullen/ros2_ws/install/mini_pupper_description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; visual mesh filename=file:///home/cullen/ros2_ws/install/mini_pupper_description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
- link lpb1: geometry collision mesh filename=file:///home/cullen/ros2_ws/install/mini_pupper_description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; visual mesh filename=file:///home/cullen/ros2_ws/install/mini_pupper_description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
- link lpb2: geometry collision mesh filename=file:///home/cullen/ros2_ws/install/mini_pupper_description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; visual mesh filename=file:///home/cullen/ros2_ws/install/mini_pupper_description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
- link lpf1: geometry collision mesh filename=file:///home/cullen/ros2_ws/install/mini_pupper_description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; visual mesh filename=file:///home/cullen/ros2_ws/install/mini_pupper_description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
- link lpf2: geometry collision mesh filename=file:///home/cullen/ros2_ws/install/mini_pupper_description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; visual mesh filename=file:///home/cullen/ros2_ws/install/mini_pupper_description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
- link rb1: geometry collision mesh filename=file:///home/cullen/ros2_ws/install/mini_pupper_description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; visual mesh filename=file:///home/cullen/ros2_ws/install/mini_pupper_description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
- link rb2: geometry collision mesh filename=file:///home/cullen/ros2_ws/install/mini_pupper_description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; visual mesh filename=file:///home/cullen/ros2_ws/install/mini_pupper_description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
- link rb3: geometry collision mesh filename=file:///home/cullen/ros2_ws/install/mini_pupper_description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; visual mesh filename=file:///home/cullen/ros2_ws/install/mini_pupper_description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
- link rbfoot: geometry collision mesh filename=file:///home/cullen/ros2_ws/install/mini_pupper_description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; visual mesh filename=file:///home/cullen/ros2_ws/install/mini_pupper_description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
- link rf1: geometry collision mesh filename=file:///home/cullen/ros2_ws/install/mini_pupper_description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; visual mesh filename=file:///home/cullen/ros2_ws/install/mini_pupper_description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
- link rf2: geometry collision mesh filename=file:///home/cullen/ros2_ws/install/mini_pupper_description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; visual mesh filename=file:///home/cullen/ros2_ws/install/mini_pupper_description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
- link rf3: geometry collision mesh filename=file:///home/cullen/ros2_ws/install/mini_pupper_description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; visual mesh filename=file:///home/cullen/ros2_ws/install/mini_pupper_description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
- link rffoot: geometry collision mesh filename=file:///home/cullen/ros2_ws/install/mini_pupper_description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; visual mesh filename=file:///home/cullen/ros2_ws/install/mini_pupper_description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
- link rpb1: geometry collision mesh filename=file:///home/cullen/ros2_ws/install/mini_pupper_description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; visual mesh filename=file:///home/cullen/ros2_ws/install/mini_pupper_description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
- link rpb2: geometry collision mesh filename=file:///home/cullen/ros2_ws/install/mini_pupper_description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; visual mesh filename=file:///home/cullen/ros2_ws/install/mini_pupper_description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
- link rpf1: geometry collision mesh filename=file:///home/cullen/ros2_ws/install/mini_pupper_description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; visual mesh filename=file:///home/cullen/ros2_ws/install/mini_pupper_description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
- link rpf2: geometry collision mesh filename=file:///home/cullen/ros2_ws/install/mini_pupper_description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; visual mesh filename=file:///home/cullen/ros2_ws/install/mini_pupper_description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
- link yellow_plate: geometry collision mesh filename=file:///home/cullen/ros2_ws/install/mini_pupper_description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; visual mesh filename=file:///home/cullen/ros2_ws/install/mini_pupper_description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
Joints:
- added joint base_link_to_base_inertia: type fixed, parent base_link, child base_inertia, origin xyz=0 0 0 rpy=0 0 0

Commit message: clean up dirty file path

File: urdf/mini_pupper_description.urdf (robot description, URDF)
Before this commit: robot mini-pupper, 39 links, 38 joints
Links:
- link base_link: geometry collision mesh filename=file://$(find mini_pupper_description)/meshes/base_link.STL; visual mesh filename=file://$(find mini_pupper_description)/meshes/base_link.STL
- link camera_link: geometry collision box size=0.02505 0.09 0.025; visual mesh filename=file://$(find mini_pupper_description)/meshes/d435.dae
- link lb1: geometry collision mesh filename=file://$(find mini_pupper_description)/meshes/lb1.STL; visual mesh filename=file://$(find mini_pupper_description)/meshes/lb1.STL
- link lb2: geometry collision mesh filename=file://$(find mini_pupper_description)/meshes/lb2.STL; visual mesh filename=file://$(find mini_pupper_description)/meshes/lb2.STL
- link lb3: geometry collision mesh filename=file://$(find mini_pupper_description)/meshes/lb3.STL; visual mesh filename=file://$(find mini_pupper_description)/meshes/lb3.STL
- link lbfoot: geometry collision mesh filename=file://$(find mini_pupper_description)/meshes/lbfoot.STL; visual mesh filename=file://$(find mini_pupper_description)/meshes/lbfoot.STL
- link lf1: geometry collision mesh filename=file://$(find mini_pupper_description)/meshes/lf1.STL; visual mesh filename=file://$(find mini_pupper_description)/meshes/lf1.STL
- link lf2: geometry collision mesh filename=file://$(find mini_pupper_description)/meshes/lf2.STL; visual mesh filename=file://$(find mini_pupper_description)/meshes/lf2.STL
- link lf3: geometry collision mesh filename=file://$(find mini_pupper_description)/meshes/lf3.STL; visual mesh filename=file://$(find mini_pupper_description)/meshes/lf3.STL
- link lffoot: geometry collision mesh filename=file://$(find mini_pupper_description)/meshes/lffoot.STL; visual mesh filename=file://$(find mini_pupper_description)/meshes/lffoot.STL
- link lidar: geometry collision mesh filename=file://$(find mini_pupper_description)/meshes/lidar.STL; visual mesh filename=file://$(find mini_pupper_description)/meshes/lidar.STL
- link lpb1: geometry collision mesh filename=file://$(find mini_pupper_description)/meshes/lpb1.STL; visual mesh filename=file://$(find mini_pupper_description)/meshes/lpb1.STL
- link lpb2: geometry collision mesh filename=file://$(find mini_pupper_description)/meshes/lpb2.STL; visual mesh filename=file://$(find mini_pupper_description)/meshes/lpb2.STL
- link lpf1: geometry collision mesh filename=file://$(find mini_pupper_description)/meshes/lpf1.STL; visual mesh filename=file://$(find mini_pupper_description)/meshes/lpf1.STL
- link lpf2: geometry collision mesh filename=file://$(find mini_pupper_description)/meshes/lpf2.STL; visual mesh filename=file://$(find mini_pupper_description)/meshes/lpf2.STL
- link rb1: geometry collision mesh filename=file://$(find mini_pupper_description)/meshes/rb1.STL; visual mesh filename=file://$(find mini_pupper_description)/meshes/rb1.STL
- link rb2: geometry collision mesh filename=file://$(find mini_pupper_description)/meshes/rb2.STL; visual mesh filename=file://$(find mini_pupper_description)/meshes/rb2.STL
- link rb3: geometry collision mesh filename=file://$(find mini_pupper_description)/meshes/rb3.STL; visual mesh filename=file://$(find mini_pupper_description)/meshes/rb3.STL
- link rbfoot: geometry collision mesh filename=file://$(find mini_pupper_description)/meshes/rbfoot.STL; visual mesh filename=file://$(find mini_pupper_description)/meshes/rbfoot.STL
- link rf1: geometry collision mesh filename=file://$(find mini_pupper_description)/meshes/rf1.STL; visual mesh filename=file://$(find mini_pupper_description)/meshes/rf1.STL
- link rf2: geometry collision mesh filename=file://$(find mini_pupper_description)/meshes/rf2.STL; visual mesh filename=file://$(find mini_pupper_description)/meshes/rf2.STL
- link rf3: geometry collision mesh filename=file://$(find mini_pupper_description)/meshes/rf3.STL; visual mesh filename=file://$(find mini_pupper_description)/meshes/rf3.STL
- link rffoot: geometry collision mesh filename=file://$(find mini_pupper_description)/meshes/rffoot.STL; visual mesh filename=file://$(find mini_pupper_description)/meshes/rffoot.STL
- link rpb1: geometry collision mesh filename=file://$(find mini_pupper_description)/meshes/rpb1.STL; visual mesh filename=file://$(find mini_pupper_description)/meshes/rpb1.STL
- link rpb2: geometry collision mesh filename=file://$(find mini_pupper_description)/meshes/rpb2.STL; visual mesh filename=file://$(find mini_pupper_description)/meshes/rpb2.STL
- link rpf1: geometry collision mesh filename=file://$(find mini_pupper_description)/meshes/rpf1.STL; visual mesh filename=file://$(find mini_pupper_description)/meshes/rpf1.STL
- link rpf2: geometry collision mesh filename=file://$(find mini_pupper_description)/meshes/rpf2.STL; visual mesh filename=file://$(find mini_pupper_description)/meshes/rpf2.STL
- link yellow_plate: geometry collision mesh filename=file://$(find mini_pupper_description)/meshes/yellow_plate.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; visual mesh filename=file://$(find mini_pupper_description)/meshes/yellow_plate.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
