Commit message: remove camera senor and fix wrong lidar sensor so for humble

File: urdf/mini_pupper_description.urdf.xacro (robot description, xacro)
@@ -4,5 +4,4 @@
      For more information, please see http://wiki.ros.org/sw_urdf_exporter -->
 <robot name="mini-pupper" xmlns:xacro="http://ros.org/wiki/xacro">
-  <xacro:include filename="$(find mini_pupper_description)/urdf/_d435.urdf.xacro" />
   <link name="base_link">
     <visual>
@@ -1758,7 +1757,10 @@
         </noise>
       </ray>
-      <plugin filename="libgazebo_ros_laser.so" name="gazebo_ros_hokuyo_controller">
-        <topicName>scan</topicName>
-        <frameName>lidar</frameName>
+      <plugin filename="libgazebo_ros_ray_sensor.so" name="gazebo_ros_lidar_controller">
+        <ros>
+          <argument>~/out:=/scan</argument>
+        </ros>
+        <output_type>sensor_msgs/LaserScan</output_type>
+        <frame_name>lidar</frame_name>
       </plugin>
     </sensor>
@@ -1806,6 +1808,3 @@
     <child link="imu_link"/>
   </joint>
-  <xacro:sensor_d435 parent="base_link">
-  <origin xyz="0.08 0.0 0.07" rpy="0 0 0" />
-  </xacro:sensor_d435>
 </robot>

Commit message: add back camera

File: urdf/mini_pupper_description.urdf.xacro (robot description, xacro)
@@ -4,4 +4,5 @@
      For more information, please see http://wiki.ros.org/sw_urdf_exporter -->
 <robot name="mini-pupper" xmlns:xacro="http://ros.org/wiki/xacro">
+  <xacro:include filename="$(find mini_pupper_description)/urdf/_d435.urdf.xacro" />
   <link name="base_link">
     <visual>
@@ -1808,3 +1809,6 @@
     <child link="imu_link"/>
   </joint>
+  <xacro:sensor_d435 parent="base_link">
+  <origin xyz="0.08 0.0 0.07" rpy="0 0 0" />
+  </xacro:sensor_d435>
 </robot>
